File: board/board.sch (KiCad schematic (older format))
At the start: 31 parts

Commit message: Finished PCB
Parts:
- removed J?: RJ45_LEDS, symbol RJ45_LEDS
- added J1: RJ45_MAGJACK, magjack:RJ45_MAGJACK, symbol RJ45_MAGJACK
- added R10: 10k, Resistors_ThroughHole:Resistor_Horizontal_RM10mm, symbol R
- C1, C12, C13, C2, C3, C5, C6: renamed from C?; footprint (none) -> Capacitors_ThroughHole:C_Disc_D3_P2.5
- C10, C11, C4, C7, C9: renamed from C?; value 0.1nF -> 0.1uF; footprint (none) -> Capacitors_ThroughHole:C_Disc_D3_P2.5
- C8: renamed from C?; footprint (none) -> Capacitors_ThroughHole:C_Radial_D5_L6_P2.5
- IC1: renamed from IC?; footprint (none) -> Housings_DIP:DIP-14_W7.62mm
- IC2: renamed from IC?; footprint DIP-28 -> Housings_DIP:DIP-28_W7.62mm
- L1: renamed from L?; footprint (none) -> Choke_Axial_ThroughHole:Choke_Horizontal_RM10mm
- P1: renamed from P?; footprint (none) -> Pin_Headers:Pin_Header_Straight_1x02
- P2: renamed from P?; footprint (none) -> Pin_Headers:Pin_Header_Straight_1x03
- R1, R2, R3, R4, R5, R6, R7, R8, R9: renamed from R?; footprint (none) -> Resistors_ThroughHole:Resistor_Horizontal_RM10mm
- U1: renamed from U?; footprint (none) -> Housings_DIP:DIP-20_W7.62mm
- U2: renamed from U?; footprint TO-220 -> Power_Integrations:TO-220
- Y1: renamed from Y?; footprint (none) -> Crystals:Crystal_HC49-U_Vertical
Connections:
- net labels added: VCC
- wire segments 101 -> 106
Other:
- note added: "Connect 5V to the hidden pin of the 7HC245\n"
- moved on the sheet: P2, R5, R7
