File: board/board.kicad_pcb (KiCad board)
At the start: 2 copper layers, 32 parts, among them IC1 PIC16F1825, IC2 ENC28J60-I/SP, J1 RJ45_MAGJACK, P1 CONN_01X02, P2 CONN_01X03, U1 74HC245, U2 LD1117V33, Y1 25MHz

Commit message: Rest of the owl (board edition)
Parts:
- moved C1 74.7 mm to (57.1, 99.7)
- moved C10 74.7 mm to (48.3, 63.5)
- moved C11 74.7 mm to (48.3, 73.7)
- moved C12 74.7 mm to (33.0, 81.3)
- moved C13 74.7 mm to (48.3, 79.4)
- moved C2 74.7 mm to (57.1, 96.5)
- moved C3 74.7 mm to (19.7, 43.2)
- moved C4 74.7 mm to (54.6, 45.7)
- moved C5 74.7 mm to (54.6, 55.9)
- moved C6 74.7 mm to (54.6, 50.8)
- moved C7 74.7 mm to (54.6, 38.7)
- moved C8 74.7 mm to (48.3, 38.1)
- moved C9 74.7 mm to (48.3, 61.0)
- moved IC1 74.7 mm to (22.9, 40.6)
- moved IC2 74.7 mm to (34.9, 40.6)
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Routing:
- net /TPOUT+: track 43.3 -> 42.4 mm
